File: PCB/V1/Channel_0.kicad_sch (KiCad schematic)
At the start: 4 parts

Commit message: Updated PCB
Parts:
- removed C: 100nF, symbol Device:C
- removed R?: 10K, symbol Device:R
- removed R?: 100K, symbol Device:R
- removed U?: TS5A3159DCKRE4, ThermoDAQ:SOT65P210X110-6N, symbol TS5A3159DCKRE4:TS5A3159DCKRE4
- added C601: 100nF, symbol Device:C
- added R601: 10K, symbol Device:R
- added R602: 100K, symbol Device:R
- added U601: TS5A3159DCKRE4, ThermoDAQ:SOT65P210X110-6N, symbol TS5A3159DCKRE4:TS5A3159DCKRE4
Connections:
- net 3V3: now also R601.1, R602.1, U601.5
- net BIAS_Select: now also U601.6
- net CH0+: now also C601.1, U601.4
- net GND: now also C601.2, U601.2
- new net: R602.2, U601.1
- new net: R601.2, U601.3
