File: PCB/V1/Channel_2.kicad_sch (KiCad schematic)
At the start: 4 parts

Commit message: Updated PCB
Parts:
- removed C?: 100nF, symbol Device:C
- removed R?: 10K, symbol Device:R
- removed R?: 100K, symbol Device:R
- removed U?: TS5A3159DCKRE4, ThermoDAQ:SOT65P210X110-6N, symbol TS5A3159DCKRE4:TS5A3159DCKRE4
- added C801: 100nF, symbol Device:C
- added R801: 10K, symbol Device:R
- added R802: 100K, symbol Device:R
- added U801: TS5A3159DCKRE4, ThermoDAQ:SOT65P210X110-6N, symbol TS5A3159DCKRE4:TS5A3159DCKRE4
Connections:
- net 3V3: now also R801.1, R802.1, U801.5
- net BIAS_Select: now also U801.6
- net CH0+: now also C801.1, U801.4
- net GND: now also C801.2, U801.2
- new net: R802.2, U801.1
- new net: R801.2, U801.3
