File: PCB/V1/Channel_3.kicad_sch (KiCad schematic)
At the start: 4 parts, among them U1101 TS5A3159DCKRE4

Commit message: Updated PCB
Parts:
- removed C1101: 100nF, symbol Device:C
- removed R1101: 10K, symbol Device:R
- removed R1102: 100K, symbol Device:R
- removed U1101: TS5A3159DCKRE4, ThermoDAQ:SOT65P210X110-6N, symbol TS5A3159DCKRE4:TS5A3159DCKRE4
- added C901: 100nF, symbol Device:C
- added R901: 10K, symbol Device:R
- added R902: 100K, symbol Device:R
- added U901: TS5A3159DCKRE4, ThermoDAQ:SOT65P210X110-6N, symbol TS5A3159DCKRE4:TS5A3159DCKRE4
Connections:
- net 3V3: now also R901.1, R902.1, U901.5
- net BIAS_Select: now also U901.6
- net CH0+: now also C901.1, U901.4
- net GND: now also C901.2, U901.2
- new net: R902.2, U901.1
- new net: R901.2, U901.3
