File: PCB/V1/Channel_4.kicad_sch (KiCad schematic)
At the start: 4 parts

Commit message: Updated PCB
Parts:
- removed C?: 100nF, symbol Device:C
- removed R?: 10K, symbol Device:R
- removed R?: 100K, symbol Device:R
- removed U?: TS5A3159DCKRE4, ThermoDAQ:SOT65P210X110-6N, symbol TS5A3159DCKRE4:TS5A3159DCKRE4
- added C1001: 100nF, symbol Device:C
- added R1001: 10K, symbol Device:R
- added R1002: 100K, symbol Device:R
- added U1001: TS5A3159DCKRE4, ThermoDAQ:SOT65P210X110-6N, symbol TS5A3159DCKRE4:TS5A3159DCKRE4
Connections:
- net 3V3: now also R1001.1, R1002.1, U1001.5
- net BIAS_Select: now also U1001.6
- net CH0+: now also C1001.1, U1001.4
- net GND: now also C1001.2, U1001.2
- new net: R1002.2, U1001.1
- new net: R1001.2, U1001.3
