File: PCB/V1/Channel_5.kicad_sch (KiCad schematic)
At the start: 4 parts

Commit message: Updated PCB
Parts:
- gave numbers to parts that had none: 4
Changed lines of the file:
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@@
 		(dnp no)
 		(fields_autoplaced yes)
-		(property "Reference" "C?"
+		(property "Reference" "C1101"
 			(at 154.94 116.8399 0)
 			(effects
@@
 			(project "V1"
 				(path "/b40ca3c0-cc7e-4fec-b4a7-67870c2202cb/6de35d57-34d9-4167-a2f8-5e880158e4d5"
-					(reference "C?")
+					(reference "C1101")
 					(unit 1)
 				)
 				(path "/b40ca3c0-cc7e-4fec-b4a7-67870c2202cb/b34d3759-fa61-425d-a208-8f586940ad14"
-					(reference "C1601")
+					(reference "C1801")
 					(unit 1)
 				)
@@
 		(dnp no)
 		(fields_autoplaced yes)
-		(property "Reference" "U?"
+		(property "Reference" "U1101"
 			(at 162.56 82.5499 90)
 			(effects
@@
 			(project "V1"
 				(path "/b40ca3c0-cc7e-4fec-b4a7-67870c2202cb/6de35d57-34d9-4167-a2f8-5e880158e4d5"
-					(reference "U?")
+					(reference "U1101")
 					(unit 1)
 				)
 				(path "/b40ca3c0-cc7e-4fec-b4a7-67870c2202cb/b34d3759-fa61-425d-a208-8f586940ad14"
-					(reference "U1601")
+					(reference "U1801")
 					(unit 1)
 				)
@@
 		(on_board yes)
 		(dnp no)
-		(property "Reference" "R?"
+		(property "Reference" "R1101"
 			(at 148.59 57.1499 0)
 			(effects
@@
 			(project "V1"
 				(path "/b40ca3c0-cc7e-4fec-b4a7-67870c2202cb/6de35d57-34d9-4167-a2f8-5e880158e4d5"
-					(reference "R?")
+					(reference "R1101")
 					(unit 1)
 				)
 				(path "/b40ca3c0-cc7e-4fec-b4a7-67870c2202cb/b34d3759-fa61-425d-a208-8f586940ad14"
-					(reference "R1601")
+					(reference "R1801")
 					(unit 1)
 				)
@@
 		(dnp no)
 		(fields_autoplaced yes)
-		(property "Reference" "#PWR?"
+		(property "Reference" "#PWR01102"
 			(at 175.26 81.28 0)
 			(effects
@@
 			(project "V1"
 				(path "/b40ca3c0-cc7e-4fec-b4a7-67870c2202cb/6de35d57-34d9-4167-a2f8-5e880158e4d5"
-					(reference "#PWR?")
+					(reference "#PWR01102")
 					(unit 1)
 				)
 				(path "/b40ca3c0-cc7e-4fec-b4a7-67870c2202cb/b34d3759-fa61-425d-a208-8f586940ad14"
-					(reference "#PWR01602")
+					(reference "#PWR01802")
 					(unit 1)
 				)
@@
 		(dnp no)
 		(fields_autoplaced yes)
-		(property "Reference" "#PWR?"
+		(property "Reference" "#PWR01101"
 			(at 151.13 135.89 0)
 			(effects
@@
 			(project "V1"
 				(path "/b40ca3c0-cc7e-4fec-b4a7-67870c2202cb/6de35d57-34d9-4167-a2f8-5e880158e4d5"
-					(reference "#PWR?")
+					(reference "#PWR01101")
 					(unit 1)
 				)
 				(path "/b40ca3c0-cc7e-4fec-b4a7-67870c2202cb/b34d3759-fa61-425d-a208-8f586940ad14"
-					(reference "#PWR01601")
+					(reference "#PWR01801")
 					(unit 1)
 				)
@@
 		(on_board yes)
 		(dnp no)
-		(property "Reference" "R?"
+		(property "Reference" "R1102"
 			(at 158.75 57.1499 0)
 			(effects
@@
 			(project "V1"
 				(path "/b40ca3c0-cc7e-4fec-b4a7-67870c2202cb/6de35d57-34d9-4167-a2f8-5e880158e4d5"
-					(reference "R?")
+					(reference "R1102")
 					(unit 1)
 				)
 				(path "/b40ca3c0-cc7e-4fec-b4a7-67870c2202cb/b34d3759-fa61-425d-a208-8f586940ad14"
-					(reference "R1602")
-					(unit 1)
-				)
+					(reference "R1802")
+					(unit 1)
+				)
