File: PCB/V1/Channel_6.kicad_sch (KiCad schematic)
At the start: 4 parts

Commit message: Updated PCB
Parts:
- removed C?: 100nF, symbol Device:C
- removed R?: 10K, symbol Device:R
- removed R?: 100K, symbol Device:R
- removed U?: TS5A3159DCKRE4, ThermoDAQ:SOT65P210X110-6N, symbol TS5A3159DCKRE4:TS5A3159DCKRE4
- added C1201: 100nF, symbol Device:C
- added R1201: 10K, symbol Device:R
- added R1202: 100K, symbol Device:R
- added U1201: TS5A3159DCKRE4, ThermoDAQ:SOT65P210X110-6N, symbol TS5A3159DCKRE4:TS5A3159DCKRE4
Connections:
- net 3V3: now also R1201.1, R1202.1, U1201.5
- net BIAS_Select: now also U1201.6
- net CH0+: now also C1201.1, U1201.4
- net GND: now also C1201.2, U1201.2
- new net: R1201.2, U1201.3
- new net: R1202.2, U1201.1
