File: PCB/V1/Channel_7.kicad_sch (KiCad schematic)
At the start: 4 parts, among them U401 TS5A3159DCKRE4

Commit message: Updated PCB
Parts:
- removed C401: 100nF, symbol Device:C
- removed R401: 10K, symbol Device:R
- removed R402: 100K, symbol Device:R
- removed U401: TS5A3159DCKRE4, ThermoDAQ:SOT65P210X110-6N, symbol TS5A3159DCKRE4:TS5A3159DCKRE4
- added C1301: 100nF, symbol Device:C
- added R1301: 10K, symbol Device:R
- added R1302: 100K, symbol Device:R
- added U1301: TS5A3159DCKRE4, ThermoDAQ:SOT65P210X110-6N, symbol TS5A3159DCKRE4:TS5A3159DCKRE4
Connections:
- net 3V3: now also R1301.1, R1302.1, U1301.5
- net BIAS_Select: now also U1301.6
- net CH0+: now also C1301.1, U1301.4
- net GND: now also C1301.2, U1301.2
- new net: R1302.2, U1301.1
- new net: R1301.2, U1301.3
