File: PCB/V1/Channel_9.kicad_sch (KiCad schematic)
At the start: 4 parts, among them U1001 TS5A3159DCKRE4

Commit message: Updated PCB
Parts:
- removed C1001: 100nF, symbol Device:C
- removed R1001: 10K, symbol Device:R
- removed R1002: 100K, symbol Device:R
- removed U1001: TS5A3159DCKRE4, ThermoDAQ:SOT65P210X110-6N, symbol TS5A3159DCKRE4:TS5A3159DCKRE4
- added C1501: 100nF, symbol Device:C
- added R1501: 10K, symbol Device:R
- added R1502: 100K, symbol Device:R
- added U1501: TS5A3159DCKRE4, ThermoDAQ:SOT65P210X110-6N, symbol TS5A3159DCKRE4:TS5A3159DCKRE4
Connections:
- net 3V3: now also R1501.1, R1502.1, U1501.5
- net BIAS_Select: now also U1501.6
- net CH0+: now also C1501.1, U1501.4
- net GND: now also C1501.2, U1501.2
- new net: R1502.2, U1501.1
- new net: R1501.2, U1501.3
