File: PCB/V1/V1.kicad_sch (KiCad schematic)
At the start: 16 parts, among them J101 Conn_01x02, J102 Conn_01x02, J103 Conn_01x02, J104 Conn_01x02, J105 Conn_01x02, J106 Conn_01x02, J107 Conn_01x02, J108 Conn_01x04

Commit message: Updated PCB
Parts:
- added C101: 10nF, symbol Device:C
- added R101: 1M, symbol Device:R
- gave numbers to parts that had none: 8
- renumbered J108 to J101, J101 to J110, J102 to J111, J103 to J112, J104 to J113, J105 to J114, J106 to J115, J107 to J116
Connections:
- net GND: now also J101.4 (Pin_4), J102.A1 (GND), J102.A12 (GND), J102.B1 (GND), J102.B12 (GND), C101.2, R101.1
- net at J102.S1 (SHIELD): now also C101.1, R101.2
- net Power_Section/RS485_VBUSS: now reaches J101.1 (Pin_1)
- net RS485_Transceiver/RS485+: now reaches J101.2 (Pin_2)
- net RS485_Transceiver/RS485-: now reaches J101.3 (Pin_3)
- net Channel_0/CH0+ renamed Channel_0/CH0
- net Channel_1/CH0+ renamed Channel_1/CH1
- net Channel_10/CH0+ renamed Channel_10/CH10
- net Channel_11/CH0+ renamed Channel_11/CH11
- net Channel_12/CH0+ renamed Channel_12/CH12
- net Channel_13/CH0+ renamed Channel_13/CH13
- net Channel_2/CH0+ renamed Channel_2/CH2
- net Channel_3/CH0+ renamed Channel_3/CH3
- net Channel_4/CH0+ renamed Channel_4/CH4
- net Channel_5/CH0+ renamed Channel_5/CH5
- net Channel_6/CH0+ renamed Channel_6/CH6
- net Channel_7/CH0+ renamed Channel_7/CH7
- net Channel_8/CH0+ renamed Channel_8/CH8
- net Channel_9/CH0+ renamed Channel_9/CH9
Other:
- added sheet RS485_Transceiver (RS485_Transceiver.kicad_sch)
- sheet Channel_0 ports: added CH0; removed CH0+
- sheet Channel_1 ports: added CH1; removed CH0+
- sheet Channel_10 ports: added CH10, TH10; removed CH0+, TH3
- sheet Channel_11 ports: added CH11, TH11; removed CH0+, TH4
- sheet Channel_12 ports: added CH12, TH12; removed CH0+, TH5
- sheet Channel_13 ports: added CH13, TH13; removed CH0+, TH6
- sheet Channel_2 ports: added CH2; removed CH0+
- sheet Channel_3 ports: added CH3; removed CH0+
- sheet Channel_4 ports: added CH4; removed CH0+
- sheet Channel_5 ports: added CH5; removed CH0+
- sheet Channel_6 ports: added CH6; removed CH0+
- sheet Channel_7 ports: added CH7, TH7; removed CH0+, TH0
- sheet Channel_8 ports: added CH8, TH8; removed CH0+, TH1
- sheet Channel_9 ports: added CH9, TH9; removed CH0+, TH2
- sheet MCU ports: added UART1_RX, UART1_TX; removed none
- sheet Power_Section ports: added RS485_VBUSS; removed none
- moved on the sheet: J101
